Commit message: Car Commit

File: proj_robo/src/robot_description/robot/robot.urdf (robot description, URDF)
Before this commit: robot yn_robot, 11 links, 10 joints
Links:
- link velodyne: geometry collision sphere radius=0; visual mesh filename=package://velodyne_description/meshes/VLP16_scan.dae
Joints:
- joint velodyne_base_mount_joint: origin xyz=0 0 -0.4 rpy=0 3.141592653589793 0 -> xyz=0 0 2 rpy=0 3.141592653589793 0

File: proj_robo/src/robot_description/robot/robot.urdf.xacro (robot description, xacro)
@@ -8,4 +8,8 @@
   <xacro:include filename="$(find velodyne_description)/urdf/VLP-16.urdf.xacro"/>
   <xacro:include filename="$(find robot_description)/urdf/IMU/IMU.urdf.xacro"/>
+  <xacro:arg name="gpu" default="false"/>
+  <xacro:property name="gpu" value="$(arg gpu)" />
+  <xacro:arg name="organize_cloud" default="false"/>
+  <xacro:property name="organize_cloud" value="$(arg organize_cloud)" />
   <!-- =============== Link & Joint =============== -->
   <!-- Base Footprint -->
@@ -47,6 +51,6 @@
   </xacro:rear_wheel_v0>
   <!--  Velodyne -->
-  <xacro:VLP-16 parent="base_link" name="velodyne" topic="/points_raw" hz="10" samples="440">
-	<origin xyz="0 0 -0.4" rpy="0 ${M_PI} 0"/>
+  <xacro:VLP-16 parent="base_link" name="velodyne" topic="/points_raw" organize_cloud="${organize_cloud}" hz="10" samples="440" gpu="${gpu}">
+	<origin xyz="0 0 2" rpy="0 ${M_PI} 0"/>
   </xacro:VLP-16>
   <!-- IMU -->

File: proj_robo/src/robot_description/urdf/IMU/IMU.gazebo.xacro (robot description, xacro)
@@ -6,5 +6,5 @@
           <sensor name="imu_sensor" type="imu">
             <always_on>true</always_on>
-            <update_rate>200</update_rate>
+            <update_rate>500</update_rate>
             <visualize>true</visualize>
             <topic>__default_topic__</topic>
@@ -14,5 +14,5 @@
                 <update_rate>0</update_rate>
                 <bodyName>imu_link</bodyName>
-                <updateRateHZ>200.0</updateRateHZ>
+                <updateRateHZ>500.0</updateRateHZ>
                 <gaussianNoise>0.0</gaussianNoise>
                 <xyzOffset>0 0 0</xyzOffset>

File: proj_robo/src/robot_gazebo/urdf/robot.urdf (robot description, URDF)
Before this commit: robot yn_robot, 11 links, 10 joints
Links:
- link velodyne: geometry collision sphere radius=0; visual mesh filename=package://velodyne_description/meshes/VLP16_scan.dae
Joints:
- removed joint base_link_joint
- added joint footprint: type fixed, parent base_footprint, child base_link, origin xyz=0 0 0 rpy=0 0 0
